File: Hardware/Spectacle_Button_Board.brd (EAGLE design)
At the start: 44.5 x 73.7 mm, 50 parts, among them J17 AUDIO-JACK3, J19 FTDI_DEVICE, J20 AUDIO-JACK3, U1 CY8C4146LQI-S422, U2 3.3V/150mA

Commit message: Checklist edits
Routing:
- net IN_5: track 59.5 -> 67.4 mm
- net GND: track 12.6 -> 7.44 mm, vias 18 -> 22
- net IN_4: track 52.3 -> 54.6 mm
Changed lines of the file:
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@@
 <wire x1="23.495" y1="41.021" x2="24.384" y2="40.132" width="0.2032" layer="1"/>
 <wire x1="24.384" y1="40.132" x2="24.384" y2="39.334" width="0.2032" layer="1"/>
-<wire x1="24.384" y1="39.334" x2="24.38" y2="39.33" width="0.254" layer="1"/>
-<wire x1="24.13" y1="36.83" x2="24.13" y2="36.957" width="0.254" layer="1"/>
-<wire x1="24.13" y1="36.957" x2="24.892" y2="37.719" width="0.254" layer="1"/>
-<wire x1="25.38" y1="39.33" x2="25.38" y2="38.08" width="0.254" layer="1"/>
-<wire x1="25.38" y1="38.08" x2="24.13" y2="36.83" width="0.254" layer="1"/>
-<wire x1="24.384" y1="39.334" x2="24.384" y2="37.084" width="0.254" layer="1"/>
 <wire x1="24.384" y1="37.084" x2="24.13" y2="36.83" width="0.254" layer="1"/>
 <contactref element="D9" pad="3"/>
@@
 <vertex x="44.45" y="73.66"/>
 </polygon>
-<via x="23.241" y="43.434" extent="1-16" drill="0.254"/>
 <wire x1="31.026" y1="29.192" x2="31.026" y2="30.315" width="0.254" layer="1"/>
 <wire x1="31.026" y1="30.315" x2="30.861" y2="30.48" width="0.254" layer="1"/>
@@
 <contactref element="J20" pad="TIP"/>
 <contactref element="J17" pad="TIP"/>
+<via x="24.13" y="36.83" extent="1-16" drill="0.254"/>
+<wire x1="25.38" y1="39.33" x2="25.38" y2="40.239" width="0.254" layer="1"/>
+<wire x1="25.38" y1="40.239" x2="25.654" y2="40.513" width="0.254" layer="1"/>
+<via x="25.654" y="40.513" extent="1-16" drill="0.254"/>
+<via x="23.241" y="43.434" extent="1-16" drill="0.254"/>
+<via x="8.128" y="41.783" extent="1-16" drill="0.254"/>
+<via x="8.128" y="52.07" extent="1-16" drill="0.254"/>
 </signal>
 <signal name="IN_0">
@@
 <wire x1="16.24" y1="35.88" x2="17.272" y2="35.88" width="0.254" layer="1"/>
 <wire x1="17.272" y1="35.88" x2="17.587" y2="35.88" width="0.254" layer="1"/>
-<wire x1="23.368" y1="6.858" x2="23.368" y2="36.068" width="0.254" layer="16"/>
-<wire x1="23.368" y1="36.068" x2="22.86" y2="36.576" width="0.254" layer="16"/>
-<wire x1="22.86" y1="36.576" x2="17.272" y2="36.576" width="0.254" layer="16"/>
+<wire x1="23.368" y1="6.858" x2="23.368" y2="35.306" width="0.254" layer="16"/>
 <via x="17.272" y="36.576" extent="1-16" drill="0.254"/>
 <wire x1="17.272" y1="36.576" x2="17.272" y2="35.88" width="0.254" layer="1"/>
@@
 <wire x1="23.622" y1="6.604" x2="23.368" y2="6.858" width="0.254" layer="16"/>
 <wire x1="31.58" y1="7.08" x2="40.83" y2="7.08" width="0.254" layer="1"/>
+<wire x1="17.272" y1="36.576" x2="21.336" y2="36.576" width="0.254" layer="16"/>
+<wire x1="21.336" y1="36.576" x2="23.368" y2="38.608" width="0.254" layer="16"/>
+<wire x1="23.368" y1="38.608" x2="25.654" y2="38.608" width="0.254" layer="16"/>
+<wire x1="25.654" y1="38.608" x2="26.289" y2="37.973" width="0.254" layer="16"/>
+<wire x1="26.289" y1="37.973" x2="26.289" y2="36.576" width="0.254" layer="16"/>
+<wire x1="26.289" y1="36.576" x2="25.654" y2="35.941" width="0.254" layer="16"/>
+<wire x1="25.654" y1="35.941" x2="24.003" y2="35.941" width="0.254" layer="16"/>
+<wire x1="24.003" y1="35.941" x2="23.368" y2="35.306" width="0.254" layer="16"/>
 </signal>
 <signal name="IN_4">
@@
 <wire x1="18.669" y1="36.068" x2="21.618" y2="36.068" width="0.254" layer="1"/>
 <wire x1="21.618" y1="36.068" x2="21.63" y2="36.08" width="0.254" layer="1"/>
-<wire x1="27.178" y1="16.383" x2="27.178" y2="37.338" width="0.254" layer="16"/>
-<wire x1="27.178" y1="37.338" x2="26.797" y2="37.719" width="0.254" layer="16"/>
-<wire x1="26.797" y1="37.719" x2="17.907" y2="37.719" width="0.254" layer="16"/>
+<wire x1="27.178" y1="16.383" x2="27.178" y2="38.735" width="0.254" layer="16"/>
 <wire x1="17.907" y1="37.719" x2="17.846" y2="37.78" width="0.254" layer="16"/>
 <via x="17.846" y="37.78" extent="1-16" drill="0.254"/>
@@
 <wire x1="40.259" y1="17.272" x2="39.402" y2="17.272" width="0.254" layer="1"/>
 <wire x1="39.402" y1="17.272" x2="39.37" y2="17.24" width="0.254" layer="1"/>
+<wire x1="17.907" y1="37.719" x2="21.082" y2="37.719" width="0.254" layer="16"/>
+<wire x1="21.082" y1="37.719" x2="22.86" y2="39.497" width="0.254" layer="16"/>
+<wire x1="22.86" y1="39.497" x2="26.416" y2="39.497" width="0.254" layer="16"/>
+<wire x1="26.416" y1="39.497" x2="27.178" y2="38.735" width="0.254" layer="16"/>
 </signal>
 <signal name="IN_6">
@@
 <contactref element="C4" pad="1"/>
 <wire x1="27.432" y1="41.457" x2="27.432" y2="40.64" width="0.254" layer="1"/>
-<wire x1="27.432" y1="40.64" x2="27.178" y2="40.386" width="0.254" layer="1"/>
-<wire x1="27.178" y1="40.386" x2="26.162" y2="40.386" width="0.254" layer="1"/>
-<wire x1="26.162" y1="40.386" x2="25.88" y2="40.104" width="0.254" layer="1"/>
-<wire x1="25.88" y1="39.33" x2="25.88" y2="40.104" width="0.254" layer="1"/>
+<wire x1="25.88" y1="39.33" x2="25.88" y2="39.85" width="0.254" layer="1"/>
+<wire x1="25.88" y1="39.85" x2="26.035" y2="40.005" width="0.254" layer="1"/>
+<wire x1="26.035" y1="40.005" x2="26.797" y2="40.005" width="0.254" layer="1"/>
+<wire x1="26.797" y1="40.005" x2="27.432" y2="40.64" width="0.254" layer="1"/>
 </signal>
 <signal name="XRES">
@@
 <wire x1="40.132" y1="45.72" x2="39.37" y2="44.958" width="0.254" layer="1"/>
 <wire x1="39.37" y1="44.958" x2="39.37" y2="39.751" width="0.254" layer="1"/>
-<wire x1="39.37" y1="39.751" x2="38.227" y2="38.608" width="0.254" layer="1"/>
-<wire x1="38.227" y1="38.608" x2="29.591" y2="38.608" width="0.254" layer="1"/>
-<wire x1="29.591" y1="38.608" x2="28.575" y2="38.608" width="0.254" layer="1"/>
-<wire x1="28.575" y1="38.608" x2="26.658" y2="38.608" width="0.254" layer="1"/>
-<wire x1="26.658" y1="38.608" x2="26.63" y2="38.58" width="0.254" layer="1"/>
-<wire x1="24.853" y1="47.879" x2="27.813" y2="47.879" width="0.254" layer="1"/>
-<wire x1="27.813" y1="47.879" x2="28.575" y2="47.117" width="0.254" layer="1"/>
-<via x="28.575" y="47.117" extent="1-16" drill="0.254"/>
-<wire x1="28.575" y1="47.117" x2="28.575" y2="40.132" width="0.254" layer="16"/>
+<wire x1="39.37" y1="39.751" x2="38.199" y2="38.58" width="0.254" layer="1"/>
 <via x="28.575" y="40.132" extent="1-16" drill="0.254"/>
-<wire x1="28.575" y1="40.132" x2="28.575" y2="38.608" width="0.254" layer="1"/>
-<wire x1="29.426" y1="33.292" x2="29.426" y2="38.443" width="0.254" layer="1"/>
-<wire x1="29.426" y1="38.443" x2="29.591" y2="38.608" width="0.254" layer="1"/>
+<wire x1="24.853" y1="47.879" x2="28.575" y2="47.879" width="0.254" layer="1"/>
+<via x="28.575" y="47.879" extent="1-16" drill="0.254"/>
+<wire x1="28.575" y1="47.879" x2="28.575" y2="40.132" width="0.254" layer="16"/>
+<wire x1="26.63" y1="38.58" x2="28.575" y2="38.58" width="0.254" layer="1"/>
+<wire x1="28.575" y1="38.58" x2="29.337" y2="38.58" width="0.254" layer="1"/>
+<wire x1="29.337" y1="38.58" x2="38.199" y2="38.58" width="0.254" layer="1"/>
+<wire x1="29.426" y1="33.292" x2="29.426" y2="38.491" width="0.254" layer="1"/>
+<wire x1="29.426" y1="38.491" x2="29.337" y2="38.58" width="0.254" layer="1"/>
+<wire x1="28.575" y1="40.132" x2="28.575" y2="38.58" width="0.254" layer="1"/>
 </signal>
 <signal name="N$3">
